Commit message: added lidar, stereo camera, gps and imu sensors to car and updated reademe

File: mursim_description/cars/gotthard/urdf/vehicle.xacro (robot description, xacro)
@@ -1,6 +1,8 @@
 <?xml version="1.0"?>
-<robot name="gotthard" xmlns:xacro="http://www.ros.org/wiki/xacro">
+<robot name="gotthard"
+  xmlns:xacro="http://www.ros.org/wiki/xacro">
   <xacro:property name="dimensions" value="${load_yaml('$(find mursim_description)/cars/gotthard/config/dimensions.yaml')}"/>
   <xacro:property name="car_settings" value="${load_yaml('$(find mursim_description)/cars/gotthard/config/car.yaml')}"/>
+  <xacro:property name="robot_sensors" value="${load_yaml('$(find mursim_description)/cars/gotthard/config/sensors.yaml')}"/>
   <!-- Vehicle Specific Includes -->
   <xacro:include filename="$(find mursim_description)/cars/gotthard/urdf/vehicle_chassis.xacro"/>
@@ -9,4 +11,5 @@
   <xacro:include filename="$(find mursim_description)/cars/gotthard/urdf/vehicle_materials.xacro"/>
   <xacro:include filename="$(find mursim_description)/cars/gotthard/urdf/vehicle_plugins.xacro"/>
+  <xacro:include filename="$(find mursim_description)/cars/gotthard/urdf/vehicle_sensors.xacro"/>
   <!-- ################################################################## -->
   <!-- ############################# Chassis ############################ -->
@@ -22,5 +25,5 @@
   <xacro:body_right_rear_wheel/>
   <!-- ############################################################################## -->
-  <!-- #### Add the left front wheel with its joints, steering and tranmissions #### -->
+  <!-- #### Add the left front wheel with its joints, steering and tranmissions  #### -->
   <!-- ############################################################################## -->
   <xacro:body_left_front_wheel/>
@@ -32,3 +35,50 @@
   <!-- ################################### Sensors ################################## -->
   <!-- ############################################################################## -->
+  <xacro:if value="${robot_sensors['sensors']['lidar_pipeline']['enabled']}">
+    <!-- define joint and link for lidar -->
+    <xacro:lidar_pipeline/>
+    <!-- find and mount os1-64 lidar -->
+    <xacro:include filename="$(find ouster_description)/urdf/OS1-64.urdf.xacro" />
+    <OS1-64 parent="front_center_lidar_link" name="os1_sensor" hz="10" samples="1024">
+      <origin xyz="0 0 0.0" rpy="0 0 0" />
+    </OS1-64>
+  </xacro:if>
+  <xacro:if value="${robot_sensors['sensors']['stereo_pipeline']['enabled']}">
+    <!-- define joint and link for camera -->
+    <xacro:camera_device/>
+    <!-- mount stereo camera -->
+    <xacro:stereo_pipeline/>
+  </xacro:if>
+  <!-- ################################### GPS ################################## -->
+  <xacro:gps_device/>
+  <gazebo>
+    <plugin name="gps_sensor" filename="libhector_gazebo_ros_gps.so">
+      <alwaysOn>1</alwaysOn>
+      <updateRate>10.0</updateRate>
+      <bodyName>gps_link</bodyName>
+      <robotBaseFrame>base_link</robotBaseFrame>
+      <topicName>${robot_sensors['sensors']['gps']['topic_name']}</topicName>
+      <velocityTopicName>${robot_sensors['sensors']['gps']['vel_topic_name']}</velocityTopicName>
+      <drift>5.0 5.0 5.0</drift>
+      <gaussianNoise>0.1 0.1 0.1</gaussianNoise>
+      <velocityDrift>0 0 0</velocityDrift>
+      <velocityGaussianNoise>0.1 0.1 0.1</velocityGaussianNoise>
+    </plugin>
+  </gazebo>
+  <!-- ################################### IMU ################################## -->
+  <xacro:imu_device/>
+  <gazebo>
+    <plugin name="imu_controller" filename="libhector_gazebo_ros_imu.so">
+      <robotNamespace>/</robotNamespace>
+      <updateRate>100.0</updateRate>
+      <bodyName>imu_link</bodyName>
+      <topicName>${robot_sensors['sensors']['imu']['topic_name']}</topicName>
+      <accelDrift>0.005 0.005 0.005</accelDrift>
+      <accelGaussianNoise>0.005 0.005 0.005</accelGaussianNoise>
+      <rateDrift>0.005 0.005 0.005 </rateDrift>
+      <rateGaussianNoise>0.005 0.005 0.005 </rateGaussianNoise>
+      <headingDrift>0.005</headingDrift>
+      <headingGaussianNoise>0.005</headingGaussianNoise>
+    </plugin>
+  </gazebo>
 </robot>

File: mursim_description/cars/gotthard/urdf/vehicle_sensors.xacro (robot description, xacro)
@@ -1,6 +1,7 @@
 <?xml version="1.0"?>
-<robot name="gotthard" xmlns:xacro="http://www.ros.org/wiki/xacro">
-	<xacro:include filename="$(find mursim_description)/cars/gotthard/urdf/vehicle_sensors_links.xacro"/>
-    <xacro:property name="sensors" value="${sensors['sensors']}"/>
+<robot name="gotthard"
+    xmlns:xacro="http://www.ros.org/wiki/xacro">
+    <xacro:include filename="$(find mursim_description)/cars/gotthard/urdf/vehicle_sensors_links.xacro"/>
+    <xacro:property name="sensors" value="${robot_sensors['sensors']}"/>
     <xacro:macro name="lidar_pipeline">
         <!-- Sensor links and fixed joints -->
@@ -14,7 +15,7 @@
             <parent link="chassis"/>
             <child link="front_center_lidar_link"/>
-            <origin xyz="${sensors['lidar']['pos']['x']} 0.0 0.15" rpy="0 0 0"/>
+            <origin xyz="${sensors['lidar']['pos']['x']} 0.0 ${sensors['lidar']['pos']['z']}" rpy="0 0 0"/>
         </joint>
-        <gazebo>
+        <!-- <gazebo>
             <plugin name="lidar_pipeline" filename="libgazebo_cone_sensor.so">
                 <yaml_config>$(arg sensors_config_file)</yaml_config>
@@ -22,8 +23,8 @@
                 <node_name>${sensors['lidar_pipeline']['node_name']}</node_name>
             </plugin>
-        </gazebo>
+        </gazebo> -->
     </xacro:macro>
     <xacro:macro name="camera_pipeline">
-        <gazebo>
+        <!-- <gazebo>
             <plugin name="camera_pipeline" filename="libgazebo_cone_sensor.so">
                 <yaml_config>$(arg sensors_config_file)</yaml_config>
@@ -31,12 +32,64 @@
                 <node_name>${sensors['camera_pipeline']['node_name']}</node_name>
             </plugin>
-        </gazebo>
+        </gazebo> -->
     </xacro:macro>
     <xacro:macro name="stereo_pipeline">
-        <gazebo>
-            <plugin name="stereo_pipeline" filename="libgazebo_cone_sensor.so">
-                <yaml_config>$(arg sensors_config_file)</yaml_config>
-                <node_name>${sensors['stereo_pipeline']['node_name']}</node_name>
-            </plugin>
+        <!-- Stereo Camera -->
+        <gazebo reference="left_camera_frame">
+            <material>Gazebo/Orange</material>
+            <sensor type="multicamera" name="stereo_camera">
+                <update_rate>${sensors['stereo_pipeline']['rate']}</update_rate>
+                <camera name="left">
+                    <horizontal_fov>1.13</horizontal_fov>
+                    <image>
+                        <width>1920</width>
+                        <height>1200</height>
+                        <format>R8G8B8</format>
+                    </image>
+                    <clip>
+                        <near>0.02</near>
+                        <far>300</far>
+                    </clip>
+                    <noise>
+                        <type>gaussian</type>
+                        <mean>0.0</mean>
+                        <stddev>0.007</stddev>
+                    </noise>
+                </camera>
+                <camera name="right">
+                    <pose>0 -${sensors['stereo_pipeline']['camera_baseline']} 0 0 0 0</pose>
+                    <horizontal_fov>1.13</horizontal_fov>
+                    <image>
+                        <width>1920</width>
+                        <height>1200</height>
+                        <format>R8G8B8</format>
+                    </image>
+                    <clip>
+                        <near>0.02</near>
+                        <far>300</far>
+                    </clip>
+                    <noise>
+                        <type>gaussian</type>
+                        <mean>0.0</mean>
+                        <stddev>0.007</stddev>
+                    </noise>
+                </camera>
+                <plugin name="stereo_camera_controller" filename="libgazebo_ros_multicamera.so">
+                    <alwaysOn>true</alwaysOn>
+                    <updateRate>0.0</updateRate>
+                    <cameraName>${sensors['stereo_pipeline']['camera_name']}</cameraName>
+                    <imageTopicName>${sensors['stereo_pipeline']['image_topic_name']}</imageTopicName>
+                    <cameraInfoTopicName>camera_info</cameraInfoTopicName>
+                    <frameName>left_camera_optical_frame</frameName>
+                    <!--<rightFrameName>right_camera_optical_frame</rightFrameName>-->
+                    <hackBaseline>${sensors['stereo_pipeline']['camera_baseline']}</hackBaseline>
+                    <distortionK1>0.0</distortionK1>
+                    <distortionK2>0.0</distortionK2>
+                    <distortionK3>0.0</distortionK3>
+                    <distortionT1>0.0</distortionT1>
+                    <distortionT2>0.0</distortionT2>
+                    <!-- <visualize>true</visualize> -->
+                </plugin>
+            </sensor>
         </gazebo>
     </xacro:macro>

File: mursim_description/cars/gotthard/urdf/vehicle_sensors_links.xacro (robot description, xacro)
@@ -1,90 +1,102 @@
 <?xml version="1.0"?>
-<robot name="gotthard" xmlns:xacro="http://www.ros.org/wiki/xacro">
-<xacro:macro name="gps_device">
-  <joint name="gps_joint" type="fixed">
-    <axis xyz="1 0 0"/> <!-- 0 1 0 -->
-    <origin xyz="1.1 0 0.56"/>
-    <parent link="cog"/>
-    <child link="gps_link"/>
-  </joint>
-  <link name="gps_link">
-    <inertial>
-      <mass value="0.001"/>
-      <origin rpy="0 0 0" xyz="0 0 0"/>
-      <inertia ixx="0.0001" ixy="0" ixz="0" iyy="0.000001" iyz="0" izz="0.0001"/>
-    </inertial>
-    <visual>
-      <origin rpy="0 0 0" xyz="0 0 0"/>
-      <geometry>
-        <box size="0.1 0.1 0.1"/>
-      </geometry>
-    </visual>
-    <collision>
-      <origin rpy="0 0 0" xyz="0 0 0"/>
-      <geometry>
-        <box size=".1 .1 .1"/>
-      </geometry>
-    </collision>
-  </link>
-</xacro:macro>
-<xacro:macro name="imu_device">
-  <joint name="imu_joint" type="fixed">
-    <axis xyz="1 0 0"/> <!-- 0 1 0 -->
-    <origin xyz="0 0 0.02"/>
-    <parent link="cog"/>
-    <child link="imu_link"/>
-  </joint>
-  <link name="imu_link">
-    <inertial>
-      <mass value="0.001"/>
-      <origin rpy="0 0 0" xyz="0 0 0"/>
-      <inertia ixx="0.0001" ixy="0" ixz="0" iyy="0.000001" iyz="0" izz="0.0001"/>
-    </inertial>
-    <visual>
-      <origin rpy="0 0 0" xyz="0 0 0"/>
-      <geometry>
-        <box size="0.05 0.05 0.05"/>
-      </geometry>
-    </visual>
-    <collision>
-      <origin rpy="0 0 0" xyz="0 0 0"/>
-      <geometry>
-        <box size="0.05 0.05 0.05"/>
-      </geometry>
-    </collision>
-  </link>
-</xacro:macro>
-<xacro:property name="camera_link" value="-1"/>
-<xacro:property name="camera_link_x" value="0.1"/>
-<xacro:property name="camera_link_y" value="0.2"/>
-<xacro:property name="camera_link_z" value="0.1"/>
-<xacro:property name="height" value="1"/>
-<xacro:macro name="camera_device">
- <joint name="camera_joint" type="fixed">
-    <axis xyz="0 1 0" />
-    <origin xyz="${camera_link} 0 ${height}" rpy="0 0 0"/>
-    <parent link="chassis"/>
-    <child link="left_camera_frame"/>
-  </joint>
-  <link name="left_camera_frame">
-    <collision>
-      <origin xyz="0 0 0" rpy="0 0 0"/>
-      <geometry>
-        <box size="${camera_link_x} ${camera_link_y} ${camera_link_z}"/>
-      </geometry>
-    </collision>
-    <visual>
-      <origin xyz="0 0 0" rpy="0 0 0"/>
-      <geometry>
-        <box size="${camera_link_x} ${camera_link_y} ${camera_link_z}"/>
-      </geometry>
-      <material name="red"/>
-    </visual>
-    <inertial>
-      <mass value="1e-5" />
-      <origin xyz="0 0 0" rpy="0 0 0"/>
-      <inertia ixx="1e-6" ixy="0" ixz="0" iyy="1e-6" iyz="0" izz="1e-6" />
-    </inertial>
-  </link>
-</xacro:macro>
+<robot name="gotthard"
+  xmlns:xacro="http://www.ros.org/wiki/xacro">
+  <xacro:macro name="gps_device">
+    <joint name="gps_joint" type="fixed">
+      <!-- <axis xyz="1 0 0"/> -->
+      <!-- 0 1 0 -->
+      <!-- for slow-lap demo place gps and imu at cog -->
+      <!-- <origin xyz="0 0 0.05"/> -->
+      <!-- <origin xyz="1.1 0 0.56"/> -->
+      <!-- <parent link="cog"/> -->
+      <!-- <child link="gps_link"/> -->
+      <axis xyz="1 0 0"/>
+      <origin xyz="0 0 0.02"/>
+      <parent link="cog"/>
+      <child link="gps_link"/>
+    </joint>
+    <link name="gps_link">
+      <inertial>
+        <mass value="0.001"/>
+        <origin rpy="0 0 0" xyz="0 0 0"/>
+        <inertia ixx="0.0001" ixy="0" ixz="0" iyy="0.000001" iyz="0" izz="0.0001"/>
+      </inertial>
+      <visual>
+        <origin rpy="0 0 0" xyz="0 0 0"/>
+        <geometry>
+          <box size="0.1 0.1 0.1"/>
+        </geometry>
+      </visual>
+      <collision>
+        <origin rpy="0 0 0" xyz="0 0 0"/>
+        <geometry>
+          <box size=".1 .1 .1"/>
+        </geometry>
+      </collision>
+    </link>
+  </xacro:macro>
+  <xacro:macro name="imu_device">
+    <joint name="imu_joint" type="fixed">
+      <axis xyz="1 0 0"/>
+      <!-- 0 1 0 -->
+      <origin xyz="0 0 0.02"/>
+      <parent link="cog"/>
+      <child link="imu_link"/>
+    </joint>
+    <link name="imu_link">
+      <inertial>
+        <mass value="0.001"/>
+        <origin rpy="0 0 0" xyz="0 0 0"/>
+        <inertia ixx="0.0001" ixy="0" ixz="0" iyy="0.000001" iyz="0" izz="0.0001"/>
+      </inertial>
+      <visual>
+        <origin rpy="0 0 0" xyz="0 0 0"/>
+        <geometry>
+          <box size="0.05 0.05 0.05"/>
+        </geometry>
+      </visual>
+      <collision>
+        <origin rpy="0 0 0" xyz="0 0 0"/>
+        <geometry>
+          <box size="0.05 0.05 0.05"/>
+        </geometry>
+      </collision>
+    </link>
+  </xacro:macro>
+  <xacro:property name="camera_link" value="-1"/>
+  <xacro:property name="camera_link_x" value="0.1"/>
+  <!-- offset to the left of the vehicle -->
+  <xacro:property name="camera_link_y" value="0.2"/>
+  <!-- <xacro:property name="camera_link_y" value="0.2"/> -->
+  <xacro:property name="camera_link_z" value="0.1"/>
+  <xacro:property name="height" value="1"/>
+  <xacro:macro name="camera_device">
+    <joint name="camera_joint" type="fixed">
+      <axis xyz="0 1 0" />
+      <!-- TODO: offset the stereo camera by half of baseline? -->
+      <origin xyz="${camera_link} 0 ${height}" rpy="0 0 0"/>
+      <parent link="chassis"/>
+      <child link="left_camera_frame"/>
+    </joint>
+    <link name="left_camera_frame">
+      <collision>
+        <origin xyz="0 0 0" rpy="0 0 0"/>
+        <geometry>
+          <box size="${camera_link_x} ${camera_link_y} ${camera_link_z}"/>
+        </geometry>
+      </collision>
+      <visual>
+        <origin xyz="0 0 0" rpy="0 0 0"/>
+        <geometry>
+          <box size="${camera_link_x} ${camera_link_y} ${camera_link_z}"/>
+        </geometry>
+        <material name="red"/>
+      </visual>
+      <inertial>
+        <mass value="1e-5" />
+        <origin xyz="0 0 0" rpy="0 0 0"/>
+        <inertia ixx="1e-6" ixy="0" ixz="0" iyy="1e-6" iyz="0" izz="1e-6" />
+      </inertial>
+    </link>
+  </xacro:macro>
 </robot>
