Commit message: initial

File: mursim_description/cars/gotthard/urdf/vehicle_properties.xacro (robot description, xacro)
@@ -44,5 +44,5 @@
 <xacro:macro name="chassis_geometry">
   <geometry>
-    <mesh filename="package://mursim_description/cars/gotthard/mesh/chassis.stl" scale = "0.001 0.001 0.001" />
+    <mesh filename="package://mursim_description/cars/gotthard/mesh/chassis.dae" scale = "1 1 1" />
   </geometry>
 </xacro:macro>
