Commit message: removed forced blue

File: mursim_description/cars/gotthard/urdf/vehicle_chassis.xacro (robot description, xacro)
@@ -34,5 +34,4 @@
             <visual>
                 <xacro:chassis_geometry/>
-                <material name="blue"/>
             </visual>
             <inertial>
@@ -40,7 +39,4 @@
             </inertial>
         </link>
-	<gazebo reference="chassis">
-	    <material>Gazebo/Blue</material>
-	</gazebo>
     </xacro:macro>
     <xacro:macro name="body_left_rear_wheel">

Commit message: changed from position controller to effort controller, added launch file for full stack under 'slow_lap.launch'

File: mursim_description/cars/gotthard/urdf/vehicle_chassis.xacro (robot description, xacro)
@@ -109,5 +109,5 @@
             <child link="left_steering_hinge"/>
             <axis xyz="0 0 1"/>
-            <limit lower="-0.8727" upper="0.8727" effort="10000000" velocity="1000000"/>
+            <limit lower="-0.8727" upper="0.8727" effort="100000.0" velocity="100000.0"/>
         </joint>
         <link name="left_steering_hinge">
@@ -152,5 +152,5 @@
                        ${dimensions['chassis']['right_steering_hinge']['y']}
                        ${dimensions['chassis']['right_steering_hinge']['z']}" rpy="0 0 0"/>
-            <limit lower="-0.8727" upper="0.8727" effort="10000000" velocity="1000000"/>
+            <limit lower="-0.8727" upper="0.8727" effort="100000.0" velocity="100000.0"/>
         </joint>
         <link name="right_steering_hinge">

Commit message: Develop/slow lap (#3)
* changed from position controller to effort controller, added launch file for full stack under 'slow_lap.launch'

* changed from postiion_controller to effort_controller

Co-authored-by: Steven Lee <stevenlee090@hotmail.com>

File: mursim_description/cars/gotthard/urdf/vehicle_chassis.xacro (robot description, xacro)
@@ -105,5 +105,5 @@
             <child link="left_steering_hinge"/>
             <axis xyz="0 0 1"/>
-            <limit lower="-0.8727" upper="0.8727" effort="10000000" velocity="1000000"/>
+            <limit lower="-0.8727" upper="0.8727" effort="100000.0" velocity="100000.0"/>
         </joint>
         <link name="left_steering_hinge">
@@ -148,5 +148,5 @@
                        ${dimensions['chassis']['right_steering_hinge']['y']}
                        ${dimensions['chassis']['right_steering_hinge']['z']}" rpy="0 0 0"/>
-            <limit lower="-0.8727" upper="0.8727" effort="10000000" velocity="1000000"/>
+            <limit lower="-0.8727" upper="0.8727" effort="100000.0" velocity="100000.0"/>
         </joint>
         <link name="right_steering_hinge">
