Commit message: repositioned camera, fixed fov to 5mm

File: mursim_description/cars/gotthard/urdf/vehicle_sensors.xacro (robot description, xacro)
@@ -41,5 +41,6 @@
                 <update_rate>${sensors['stereo_pipeline']['rate']}</update_rate>
                 <camera name="left">
-                    <horizontal_fov>1.13</horizontal_fov>
+                    <pose>0 0.1 0 0 0 0</pose>
+                    <horizontal_fov>1</horizontal_fov>
                     <image>
                         <width>1920</width>
@@ -58,6 +59,6 @@
                 </camera>
                 <camera name="right">
-                    <pose>0 -${sensors['stereo_pipeline']['camera_baseline']} 0 0 0 0</pose>
-                    <horizontal_fov>1.13</horizontal_fov>
+                    <pose>0 -0.1 0 0 0 0</pose>
+                    <horizontal_fov>1</horizontal_fov>
                     <image>
                         <width>1920</width>

File: mursim_description/cars/gotthard/urdf/vehicle_sensors_links.xacro (robot description, xacro)
@@ -64,5 +64,5 @@
     </link>
   </xacro:macro>
-  <xacro:property name="camera_link" value="-1"/>
+  <xacro:property name="camera_link" value="-0.9"/>
   <xacro:property name="camera_link_x" value="0.1"/>
   <!-- offset to the left of the vehicle -->
