Commit message: separated 19E from the dynamic model

File: mursim_description/cars/19E-dynamic/urdf/vehicle_plugins.xacro (robot description, xacro)
@@ -1,5 +1,5 @@
 <?xml version="1.0"?>
 <robot name="19E" xmlns:xacro="http://www.ros.org/wiki/xacro">
-  <!-- ############################## STEERING #############################-->
+    <!-- STEERING -->
     <transmission name="left_steering">
 	<type>transmission_interface/SimpleTransmission</type>
@@ -22,5 +22,5 @@
 	</actuator>
     </transmission>
-  <!-- ############################## DRIVETRAIN #############################-->
+    <!-- DRIVE -->
     <transmission name="front_left_drive">
 	<type>transmission_interface/SimpleTransmission</type>
@@ -59,9 +59,10 @@
 	</actuator>
     </transmission>
-  <!-- ############################## ACUTATION #############################-->
+    <!--
     <gazebo>
-      <plugin name="gazebo_ros_control" filename="libgazebo_ros_control.so">
-          <robotNamespace>/19E/steer_drive_controller</robotNamespace>
-      </plugin>
+	<plugin name="gazebo_ros_control" filename="libgazebo_ros_control.so">
+	    <robotNamespace>/19E/steer_drive_controller</robotNamespace>
+	</plugin>
     </gazebo>
+    -->
 </robot>

File: mursim_description/cars/19E-dynamic/urdf/vehicle_sensors.xacro (robot description, xacro)
@@ -1,9 +1,20 @@
 <?xml version="1.0"?>
-<robot name="19E" xmlns:xacro="http://www.ros.org/wiki/xacro">
+<robot name="19E"
+    xmlns:xacro="http://www.ros.org/wiki/xacro">
     <xacro:include filename="$(find mursim_description)/cars/19E/urdf/vehicle_sensors_links.xacro"/>
     <xacro:property name="sensors" value="${robot_sensors['sensors']}"/>
-    <!-- ############################ LIDAR ############################# -->
-    <!-- find and mount os1-64 lidar -->
-    <xacro:macro name="lidar">
+    <xacro:macro name="lidar_pipeline">
+        <!-- Sensor links and fixed joints -->
+        <link name="front_center_lidar_link">
+            <inertial>
+                <mass value="1"/>
+                <inertia ixx="0.001" ixy="0.0" ixz="0.0" iyy="0.001" iyz="0.0" izz="0.001"/>
+            </inertial>
+        </link>
+        <joint name="front_center_lidar_joint" type="fixed">
+            <parent link="chassis"/>
+            <child link="front_center_lidar_link"/>
+            <origin xyz="${sensors['lidar']['pos']['x']} 0.0 ${sensors['lidar']['pos']['z']}" rpy="0 0 0"/>
+        </joint>
         <!-- <gazebo>
             <plugin name="lidar_pipeline" filename="libgazebo_cone_sensor.so">
@@ -14,5 +25,4 @@
         </gazebo> -->
     </xacro:macro>
-    <!-- ############################ CAMERAS ############################# -->
     <xacro:macro name="camera_pipeline">
         <!-- <gazebo>
@@ -84,48 +94,3 @@
         </gazebo>
     </xacro:macro>
-    <!-- ############################ GPS ############################# -->
-    <xacro:macro name="gps_pipeline">
-        <gazebo>
-          <plugin name="gps_sensor" filename="libhector_gazebo_ros_gps.so">
-            <alwaysOn>1</alwaysOn>
-            <updateRate>10.0</updateRate>
-            <bodyName>gps_link</bodyName>
-            <robotBaseFrame>base_link</robotBaseFrame>
-            <topicName>${robot_sensors['sensors']['gps']['topic_name']}</topicName>
-            <velocityTopicName>${robot_sensors['sensors']['gps']['vel_topic_name']}</velocityTopicName>
-            <drift>5.0 5.0 5.0</drift>
-            <gaussianNoise>0.1 0.1 0.1</gaussianNoise>
-            <velocityDrift>0 0 0</velocityDrift>
-            <velocityGaussianNoise>0.1 0.1 0.1</velocityGaussianNoise>
-          </plugin>
-        </gazebo>
-    </xacro:macro>
-    <!-- ############################ IMU ############################# -->
-    <xacro:macro name="imu_pipeline">
-        <gazebo>
-          <plugin name="imu_controller" filename="libhector_gazebo_ros_imu.so">
-            <robotNamespace>/</robotNamespace>
-            <updateRate>100.0</updateRate>
-            <bodyName>imu_link</bodyName>
-            <topicName>${robot_sensors['sensors']['imu']['topic_name']}</topicName>
-            <accelDrift>0.005 0.005 0.005</accelDrift>
-            <accelGaussianNoise>0.005 0.005 0.005</accelGaussianNoise>
-            <rateDrift>0.005 0.005 0.005 </rateDrift>
-            <rateGaussianNoise>0.005 0.005 0.005 </rateGaussianNoise>
-            <headingDrift>0.005</headingDrift>
-            <headingGaussianNoise>0.005</headingGaussianNoise>
-          </plugin>
-        </gazebo>
-    </xacro:macro>
-    <!-- ####################### GROUND TRUTH #########################-->
-    <xacro:macro name="p3d_ground_truth">
-        <gazebo>
-          <plugin name="ground_truth" filename="libgazebo_ros_p3d.so">
-            <frameName>map</frameName>
-            <bodyName>base_link</bodyName>
-            <topicName>odom</topicName>
-            <updateRate>30.0</updateRate>
-          </plugin>
-        </gazebo>
-    </xacro:macro>
 </robot>

File: mursim_description/cars/19E-dynamic/urdf/vehicle_sensors_links.xacro (robot description, xacro)
@@ -2,23 +2,4 @@
 <robot name="19E"
   xmlns:xacro="http://www.ros.org/wiki/xacro">
-  <!-- ######################## LIDAR LINKS ########################## -->
-  <xacro:macro name="lidar_pipeline">
-      <link name="front_center_lidar_link">
-          <inertial>
-              <mass value="1"/>
-              <inertia ixx="0.001" ixy="0.0" ixz="0.0" iyy="0.001" iyz="0.0" izz="0.001"/>
-          </inertial>
-      </link>
-      <joint name="front_center_lidar_joint" type="fixed">
-          <parent link="chassis"/>
-          <child link="front_center_lidar_link"/>
-          <origin xyz="${sensors['lidar_pipeline']['pos']['x']} 0.0 ${sensors['lidar_pipeline']['pos']['z']}" rpy="0 0 0"/>
-      </joint>
-      <xacro:include filename="$(find ouster_description)/urdf/OS1-64.urdf.xacro" />
-      <OS1-64 parent="front_center_lidar_link" name="os1_sensor" hz="10" samples="1024">
-        <origin xyz="0 0 0.0" rpy="0 0 0" />
-      </OS1-64>
-  </xacro:macro>
-  <!-- ######################## GPS LINKS ########################## -->
   <xacro:macro name="gps_device">
     <joint name="gps_joint" type="fixed">
@@ -38,13 +19,9 @@
       <inertial>
         <mass value="0.001"/>
-        <origin xyz="${sensors['gps']['pos']['x']}
-                     ${sensors['gps']['pos']['y']}
-                     ${sensors['gps']['pos']['z']}" rpy="0 0 0"/>
+        <origin rpy="0 0 0" xyz="0 0 0"/>
         <inertia ixx="0.0001" ixy="0" ixz="0" iyy="0.000001" iyz="0" izz="0.0001"/>
       </inertial>
       <visual>
-        <origin xyz="${sensors['gps']['pos']['x']}
-                     ${sensors['gps']['pos']['y']}
-                     ${sensors['gps']['pos']['z']}" rpy="0 0 0"/>
+        <origin rpy="0 0 0" xyz="0 0 0"/>
         <geometry>
           <box size="0.1 0.1 0.1"/>
@@ -52,8 +29,6 @@
       </visual>
       <collision>
+        <origin rpy="0 0 0" xyz="0 0 0"/>
         <geometry>
-         <origin xyz="${sensors['gps']['pos']['x']}
-                     ${sensors['gps']['pos']['y']}
-                     ${sensors['gps']['pos']['z']}" rpy="0 0 0"/>
           <box size=".1 .1 .1"/>
         </geometry>
@@ -61,5 +36,4 @@
     </link>
   </xacro:macro>
-  <!-- ######################## IMU LINKS ########################## -->
   <xacro:macro name="imu_device">
     <joint name="imu_joint" type="fixed">
@@ -73,13 +47,9 @@
       <inertial>
         <mass value="0.001"/>
-        <origin xyz="${sensors['imu']['pos']['x']}
-                     ${sensors['imu']['pos']['y']}
-                     ${sensors['imu']['pos']['z']}" rpy="0 0 0"/>
+        <origin rpy="0 0 0" xyz="0 0 0"/>
         <inertia ixx="0.0001" ixy="0" ixz="0" iyy="0.000001" iyz="0" izz="0.0001"/>
       </inertial>
       <visual>
-        <origin xyz="${sensors['imu']['pos']['x']}
-                     ${sensors['imu']['pos']['y']}
-                     ${sensors['imu']['pos']['z']}" rpy="0 0 0"/>
+        <origin rpy="0 0 0" xyz="0 0 0"/>
         <geometry>
           <box size="0.05 0.05 0.05"/>
@@ -87,7 +57,5 @@
       </visual>
       <collision>
-        <origin xyz="${sensors['imu']['pos']['x']}
-                     ${sensors['imu']['pos']['y']}
-                     ${sensors['imu']['pos']['z']}" rpy="0 0 0"/>
+        <origin rpy="0 0 0" xyz="0 0 0"/>
         <geometry>
           <box size="0.05 0.05 0.05"/>
@@ -96,5 +64,4 @@
     </link>
   </xacro:macro>
-  <!-- ######################## CAMERA LINKS ########################## -->
   <xacro:property name="camera_link" value="-1"/>
   <xacro:property name="camera_link_x" value="0.1"/>

File: mursim_description/cars/19E/urdf/vehicle.xacro (robot description, xacro)
@@ -11,36 +11,17 @@
   <xacro:include filename="$(find mursim_description)/cars/19E/urdf/vehicle_plugins.xacro"/>
   <xacro:include filename="$(find mursim_description)/cars/19E/urdf/vehicle_sensors.xacro"/>
-  <!-- ################################################################## -->
   <!-- ############################# Chassis ############################ -->
-  <!-- ################################################################## -->
   <xacro:body_chassis/>
-  <!-- ################################################################## -->
   <!-- #### Add the left rear wheel with its joints and tranmissions #### -->
-  <!-- ################################################################## -->
   <xacro:body_left_rear_wheel/>
-  <!-- ################################################################### -->
   <!-- #### Add the right rear wheel with its joints and tranmissions #### -->
-  <!-- ################################################################### -->
   <xacro:body_right_rear_wheel/>
-  <!-- ############################################################################## -->
   <!-- #### Add the left front wheel with its joints, steering and tranmissions  #### -->
-  <!-- ############################################################################## -->
   <xacro:body_left_front_wheel/>
-  <!-- ############################################################################## -->
   <!-- #### Add the right front wheel with its joints, steering and tranmissions #### -->
-  <!-- ############################################################################## -->
   <xacro:body_right_front_wheel/>
-  <!-- ############################################################################## -->
   <!-- ################################### Sensors ################################## -->
-  <!-- ############################################################################## -->
   <xacro:if value="${robot_sensors['sensors']['lidar_pipeline']['enabled']}">
-    <!-- define joint and link for lidar -->
     <xacro:lidar_pipeline/>
-    <!-- find and mount os1-64 lidar -->
-    <xacro:include filename="$(find ouster_description)/urdf/OS1-64.urdf.xacro" />
-    <OS1-64 parent="front_center_lidar_link" name="os1_sensor" hz="10" samples="1024">
-      <origin xyz="0 0 0.0" rpy="0 0 0" />
-    </OS1-64>
-  </xacro:if>
   <xacro:if value="${robot_sensors['sensors']['stereo_pipeline']['enabled']}">
     <!-- define joint and link for camera -->
@@ -50,55 +31,14 @@
   </xacro:if>
   <!-- ################################### GPS ################################## -->
-  <xacro:gps_device/>
-  <gazebo>
-    <plugin name="gps_sensor" filename="libhector_gazebo_ros_gps.so">
-      <alwaysOn>1</alwaysOn>
-      <updateRate>10.0</updateRate>
-      <bodyName>gps_link</bodyName>
-      <robotBaseFrame>base_link</robotBaseFrame>
-      <topicName>${robot_sensors['sensors']['gps']['topic_name']}</topicName>
-      <velocityTopicName>${robot_sensors['sensors']['gps']['vel_topic_name']}</velocityTopicName>
-      <drift>5.0 5.0 5.0</drift>
-      <gaussianNoise>0.1 0.1 0.1</gaussianNoise>
-      <velocityDrift>0 0 0</velocityDrift>
-      <velocityGaussianNoise>0.1 0.1 0.1</velocityGaussianNoise>
-    </plugin>
-  </gazebo>
+  <xacro:if value="${robot_sensors['sensors']['gps_pipeline']['enabled']}">
+      <xacro:gps_pipeline/>
+  </xacro:if>
   <!-- ################################### IMU ################################## -->
-  <xacro:imu_device/>
-  <gazebo>
-    <plugin name="imu_controller" filename="libhector_gazebo_ros_imu.so">
-      <robotNamespace>/</robotNamespace>
-      <updateRate>100.0</updateRate>
-      <bodyName>imu_link</bodyName>
-      <topicName>${robot_sensors['sensors']['imu']['topic_name']}</topicName>
-      <accelDrift>0.005 0.005 0.005</accelDrift>
-      <accelGaussianNoise>0.005 0.005 0.005</accelGaussianNoise>
-      <rateDrift>0.005 0.005 0.005 </rateDrift>
-      <rateGaussianNoise>0.005 0.005 0.005 </rateGaussianNoise>
-      <headingDrift>0.005</headingDrift>
-      <headingGaussianNoise>0.005</headingGaussianNoise>
-    </plugin>
-  </gazebo>
+  <xacro:if value="${robot_sensors['sensors']['imu_pipeline']['enabled']}">
+      <xacro:imu_pipeline/>
+  </xacro:if>
   <!-- ################################### P3D ################################## -->
-  <gazebo>
-    <plugin name="ground_truth" filename="libgazebo_ros_p3d.so">
-      <frameName>map</frameName>
-      <bodyName>base_link</bodyName>
-      <topicName>odom</topicName>
-      <updateRate>30.0</updateRate>
-    </plugin>
-  </gazebo>
-  <!-- ################################### TEMP ################################## -->
-  <gazebo>
-      <plugin name="mursim_physics" filename="libmursim_physics.so">
-	  <chassis>base_link</chassis>
-	  <robot_name>19E</robot_name>
-	  <base_link>base_link</base_link>
-	  <front_left_wheel>front_left_wheel_joint</front_left_wheel>
-	  <front_right_wheel>front_right_wheel_joint</front_right_wheel>
-	  <rear_left_wheel>rear_left_wheel_joint</rear_left_wheel>
-	  <rear_right_wheel>rear_right_wheel_joint</rear_right_wheel>
-      </plugin>
-  </gazebo>
+  <xacro:if value="${robot_sensors['ground_truth']['enabled']}">
+      <xacro:p3d_ground_truth/>
+  </xacro:if>
 </robot>
