Commit message: fixed lidar was not spawning correct

File: mursim_description/cars/19E-dynamic/urdf/vehicle_sensors_links.xacro (robot description, xacro)
@@ -2,4 +2,10 @@
 <robot name="19E"
   xmlns:xacro="http://www.ros.org/wiki/xacro">
+  <xacro:macro name="lidar_device">
+      <link name="front_center_lidar_link">
+          <inertial>
+              <mass value="1"/>
+              <inertia ixx="0.001" ixy="0.0" ixz="0.0" iyy="0.001" iyz="0.0" izz="0.001"/>
+  </xacro:macro>
   <xacro:macro name="gps_device">
     <joint name="gps_joint" type="fixed">

File: mursim_description/cars/19E/urdf/vehicle_sensors.xacro (robot description, xacro)
@@ -6,4 +6,5 @@
     <!-- find and mount os1-64 lidar -->
     <xacro:macro name="lidar_pipeline">
+        <xacro:lidar_device/>
         <!-- <gazebo>
             <plugin name="lidar_pipeline" filename="libgazebo_cone_sensor.so">
@@ -13,4 +14,8 @@
             </plugin>
         </gazebo> -->
+        <xacro:include filename="$(find ouster_description)/urdf/OS1-64.urdf.xacro" />
+        <OS1-64 parent="front_center_lidar_link" name="os1_sensor" hz="10" samples="1024">
+            <origin xyz="0 0 0.0" rpy="0 0 0" />
+        </OS1-64>
     </xacro:macro>
     <!-- ############################ CAMERAS ############################# -->

File: mursim_description/cars/19E/urdf/vehicle_sensors_links.xacro (robot description, xacro)
@@ -3,5 +3,5 @@
   xmlns:xacro="http://www.ros.org/wiki/xacro">
   <!-- ######################## LIDAR LINKS ########################## -->
-  <xacro:macro name="lidar_pipeline">
+  <xacro:macro name="lidar_device">
       <link name="front_center_lidar_link">
           <inertial>
@@ -15,8 +15,4 @@
           <origin xyz="${sensors['lidar_pipeline']['pos']['x']} 0.0 ${sensors['lidar_pipeline']['pos']['z']}" rpy="0 0 0"/>
       </joint>
-      <xacro:include filename="$(find ouster_description)/urdf/OS1-64.urdf.xacro" />
-      <OS1-64 parent="front_center_lidar_link" name="os1_sensor" hz="10" samples="1024">
-        <origin xyz="0 0 0.0" rpy="0 0 0" />
-      </OS1-64>
   </xacro:macro>
   <!-- ######################## GPS LINKS ########################## -->
