Commit message: base written, testing

File: mursim_description/cars/19E/urdf/vehicle.xacro (robot description, xacro)
@@ -90,3 +90,17 @@
     </plugin>
   </gazebo>
+  <!-- ################################### TEMP ################################## -->
+<!--
+  <gazebo>
+      <plugin name="mursim_physics" filename="libmursim_physics.so">
+	  <chassis>base_link</chassis>
+	  <robot_name>19E</robot_name>
+	  <base_link>base_link</base_link>
+	  <front_left_wheel>front_left_wheel_joint</front_left_wheel>
+	  <front_left_wheel>front_right_wheel_joint</front_left_wheel>
+	  <rear_left_wheel>rear_left_wheel_joint</rear_left_wheel>
+	  <rear_right_wheel>rear_right_wheel_joint</rear_right_wheel>
+      </plugin>
+  </gazebo>
+-->
 </robot>

File: mursim_description/cars/gotthard/urdf/vehicle_properties.xacro (robot description, xacro)
@@ -44,5 +44,5 @@
 <xacro:macro name="chassis_geometry">
   <geometry>
-    <mesh filename="package://mursim_description/cars/gotthard/mesh/chassis.dae" scale = "1 1 1" />
+    <mesh filename="package://mursim_description/cars/gotthard/mesh/whole_car.stl" scale = "0.001 0.001 0.001" />
   </geometry>
 </xacro:macro>

Commit message: fixed naming errors for 19E

File: mursim_description/cars/19E/urdf/vehicle.xacro (robot description, xacro)
@@ -24,4 +24,5 @@
   <xacro:if value="${robot_sensors['sensors']['lidar_pipeline']['enabled']}">
     <xacro:lidar_pipeline/>
+  </xacro:if>
   <xacro:if value="${robot_sensors['sensors']['stereo_pipeline']['enabled']}">
     <!-- define joint and link for camera -->

File: mursim_description/cars/19E/urdf/vehicle_sensors.xacro (robot description, xacro)
@@ -5,5 +5,5 @@
     <!-- ############################ LIDAR ############################# -->
     <!-- find and mount os1-64 lidar -->
-    <xacro:macro name="lidar">
+    <xacro:macro name="lidar_pipeline">
         <!-- <gazebo>
             <plugin name="lidar_pipeline" filename="libgazebo_cone_sensor.so">
@@ -86,4 +86,5 @@
     <!-- ############################ GPS ############################# -->
     <xacro:macro name="gps_pipeline">
+        <xacro:gps_device/>
         <gazebo>
           <plugin name="gps_sensor" filename="libhector_gazebo_ros_gps.so">
@@ -92,6 +93,6 @@
             <bodyName>gps_link</bodyName>
             <robotBaseFrame>base_link</robotBaseFrame>
-            <topicName>${robot_sensors['sensors']['gps']['topic_name']}</topicName>
-            <velocityTopicName>${robot_sensors['sensors']['gps']['vel_topic_name']}</velocityTopicName>
+            <topicName>${robot_sensors['sensors']['gps_pipeline']['topic_name']}</topicName>
+            <velocityTopicName>${robot_sensors['sensors']['gps_pipeline']['vel_topic_name']}</velocityTopicName>
             <drift>5.0 5.0 5.0</drift>
             <gaussianNoise>0.1 0.1 0.1</gaussianNoise>
@@ -103,4 +104,5 @@
     <!-- ############################ IMU ############################# -->
     <xacro:macro name="imu_pipeline">
+        <xacro:imu_device/>
         <gazebo>
           <plugin name="imu_controller" filename="libhector_gazebo_ros_imu.so">
@@ -108,5 +110,5 @@
             <updateRate>100.0</updateRate>
             <bodyName>imu_link</bodyName>
-            <topicName>${robot_sensors['sensors']['imu']['topic_name']}</topicName>
+            <topicName>${robot_sensors['sensors']['imu_pipeline']['topic_name']}</topicName>
             <accelDrift>0.005 0.005 0.005</accelDrift>
             <accelGaussianNoise>0.005 0.005 0.005</accelGaussianNoise>

File: mursim_description/cars/19E/urdf/vehicle_sensors_links.xacro (robot description, xacro)
@@ -38,13 +38,13 @@
       <inertial>
         <mass value="0.001"/>
-        <origin xyz="${sensors['gps']['pos']['x']}
-                     ${sensors['gps']['pos']['y']}
-                     ${sensors['gps']['pos']['z']}" rpy="0 0 0"/>
+        <origin xyz="${sensors['gps_pipeline']['pos']['x']}
+                     ${sensors['gps_pipeline']['pos']['y']}
+                     ${sensors['gps_pipeline']['pos']['z']}" rpy="0 0 0"/>
         <inertia ixx="0.0001" ixy="0" ixz="0" iyy="0.000001" iyz="0" izz="0.0001"/>
       </inertial>
       <visual>
-        <origin xyz="${sensors['gps']['pos']['x']}
-                     ${sensors['gps']['pos']['y']}
-                     ${sensors['gps']['pos']['z']}" rpy="0 0 0"/>
+        <origin xyz="${sensors['gps_pipeline']['pos']['x']}
+                     ${sensors['gps_pipeline']['pos']['y']}
+                     ${sensors['gps_pipeline']['pos']['z']}" rpy="0 0 0"/>
         <geometry>
           <box size="0.1 0.1 0.1"/>
@@ -53,7 +53,7 @@
       <collision>
         <geometry>
-         <origin xyz="${sensors['gps']['pos']['x']}
-                     ${sensors['gps']['pos']['y']}
-                     ${sensors['gps']['pos']['z']}" rpy="0 0 0"/>
+         <origin xyz="${sensors['gps_pipeline']['pos']['x']}
+                     ${sensors['gps_pipeline']['pos']['y']}
+                     ${sensors['gps_pipeline']['pos']['z']}" rpy="0 0 0"/>
           <box size=".1 .1 .1"/>
         </geometry>
@@ -73,13 +73,13 @@
       <inertial>
         <mass value="0.001"/>
-        <origin xyz="${sensors['imu']['pos']['x']}
-                     ${sensors['imu']['pos']['y']}
-                     ${sensors['imu']['pos']['z']}" rpy="0 0 0"/>
+        <origin xyz="${sensors['imu_pipeline']['pos']['x']}
+                     ${sensors['imu_pipeline']['pos']['y']}
+                     ${sensors['imu_pipeline']['pos']['z']}" rpy="0 0 0"/>
         <inertia ixx="0.0001" ixy="0" ixz="0" iyy="0.000001" iyz="0" izz="0.0001"/>
       </inertial>
       <visual>
-        <origin xyz="${sensors['imu']['pos']['x']}
-                     ${sensors['imu']['pos']['y']}
-                     ${sensors['imu']['pos']['z']}" rpy="0 0 0"/>
+        <origin xyz="${sensors['imu_pipeline']['pos']['x']}
+                     ${sensors['imu_pipeline']['pos']['y']}
+                     ${sensors['imu_pipeline']['pos']['z']}" rpy="0 0 0"/>
         <geometry>
           <box size="0.05 0.05 0.05"/>
@@ -87,7 +87,7 @@
       </visual>
       <collision>
-        <origin xyz="${sensors['imu']['pos']['x']}
-                     ${sensors['imu']['pos']['y']}
-                     ${sensors['imu']['pos']['z']}" rpy="0 0 0"/>
+        <origin xyz="${sensors['imu_pipeline']['pos']['x']}
+                     ${sensors['imu_pipeline']['pos']['y']}
+                     ${sensors['imu_pipeline']['pos']['z']}" rpy="0 0 0"/>
         <geometry>
           <box size="0.05 0.05 0.05"/>
