Commit message: fixed typo in sensor links xacro file for 19E

File: mursim_description/cars/19E/urdf/vehicle_sensors_links.xacro (robot description, xacro)
@@ -52,8 +52,8 @@
       </visual>
       <collision>
-        <geometry>
          <origin xyz="${sensors['gps_pipeline']['pos']['x']}
                      ${sensors['gps_pipeline']['pos']['y']}
                      ${sensors['gps_pipeline']['pos']['z']}" rpy="0 0 0"/>
+        <geometry>
           <box size=".1 .1 .1"/>
         </geometry>
